File: acdc_switch_supply_tryout.sch (KiCad schematic (older format))
At the start: 6 parts

Commit message: update,
Parts:
- J?: footprint (none) -> Connector_PinHeader_2.54mm:PinHeader_1x02_P2.54mm_Vertical
- TH?: footprint footprint-lib:NTC 10D-11 -> footprint-lib:10D-11
Changed lines of the file:
@@
 F 0 "TH?" V 3060 900 50  0000 C CNN
 F 1 "10D-11" V 3151 900 50  0000 C CNN
-F 2 "footprint-lib:NTC 10D-11" H 3350 950 50  0001 C CNN
+F 2 "footprint-lib:10D-11" H 3350 950 50  0001 C CNN
 F 3 "~" H 3350 950 50  0001 C CNN
 	1    3350 900
@@
 F 0 "J?" H 6078 876 50  0000 L CNN
 F 1 "LV_OUTPUT" H 6078 785 50  0000 L CNN
-F 2 "" H 6050 900 50  0001 C CNN
+F 2 "Connector_PinHeader_2.54mm:PinHeader_1x02_P2.54mm_Vertical" H 6050 900 50  0001 C CNN
 F 3 "~" H 6050 900 50  0001 C CNN
 	1    6050 900
